Commit message: [Models] eve with gripper frames

File: models/eve.urdf (robot description, URDF)
Before this commit: robot architect, 6 links, 5 joints
Links:
- added link left_gripper_frame
- added link right_gripper_frame
Joints:
- added joint left_gripper_joint: type fixed, parent arm_left_link, child left_gripper_frame, origin xyz=0.0 -0.05 -0.42 rpy=0 0.0 0
- added joint right_gripper_joint: type fixed, parent arm_right_link, child right_gripper_frame, origin xyz=0.0 0.05 -0.42 rpy=0 0.0 0

Commit message: Update and save of the fusion branch

File: models/eve.urdf (robot description, URDF)
Before this commit: robot eve, 8 links, 7 joints
Links:
- removed link head_camera_frame
- added link eve_head
- added link left_eye_camera_frame
- added link right_eye_camera_frame
Joints:
- removed joint head_camera_frame_joint
- added joint eve_head_joint: type fixed, parent head, child eve_head, origin xyz=0.19 0.0 0.24 rpy=-1.57079632679 0.0 -1.57079632679
- added joint left_eye_joint: type fixed, parent head, child left_eye_camera_frame, origin xyz=0.1 0.05 0.25 rpy=0 0 0
- added joint right_eye_joint: type fixed, parent head, child right_eye_camera_frame, origin xyz=0.1 -0.05 0.25 rpy=0 0 0

Commit message: [Doc] update with robot's sensors

File: models/eve.urdf (robot description, URDF)
Before this commit: robot eve, 10 links, 9 joints
Links:
- removed link head
- removed link left_eye_camera_frame
- removed link right_eye_camera_frame
- added link head_camera_frame
- link eve_head: geometry collision mesh filename=package://overworld/models/tutorials/Eve/eve_head.obj; visual mesh filename=package://overworld/models/tutorials/Eve/eve_head.obj
Joints:
- removed joint left_eye_joint
- removed joint right_eye_joint
- joint eve_head_joint: child eve_head -> head_camera_frame; parent head -> eve_head
- joint head_joint: child head -> eve_head
