Commit message: [models] add test models

File: models/tutorials/Frame/frame.urdf (robot description, URDF)
Before this commit: robot frame, 1 links, 0 joints
Links:
- removed link adream_walls
- added link frame_y, mass .0; collision mesh filename=package://overworld/models/tutorials/Frame/frame.obj scale=1 1 1; visual mesh filename=package://overworld/models/tutorials/Frame/frame.obj scale=1 1 1
- added link frame_z, mass .0; collision mesh filename=package://overworld/models/tutorials/Frame/frame.obj scale=1 1 1; visual mesh filename=package://overworld/models/tutorials/Frame/frame_z.dae scale=1 1 1
Joints:
- added joint frame_link: type fixed, parent frame_y, child frame_z, origin xyz=-1 1 0 rpy=0 0 0
