Commit message: [Engine] Obj and Stl loaders

File: models/adream/adream.urdf (robot description, URDF)
Before this commit: robot adream, 8 links, 7 joints
Links:
- link adream_window_h10_1: geometry visual mesh filename=package://overworld/models/adream/window_h10_1.stl scale=1 1 1

Commit message: [Models] reduce textures size

File: models/adream/adream.urdf (robot description, URDF)
Before this commit: robot adream, 8 links, 7 joints
Links:
- removed link adream_floor
- added link adream_floor_expe, mass .0; collision mesh filename=package://overworld/models/adream/floor_expe_collision.obj scale=1 1 1; visual mesh filename=package://overworld/models/adream/floor_expe.obj scale=1 1 1
- added link adream_floor_hall, mass .0; collision mesh filename=package://overworld/models/adream/floor_hall_collision.obj scale=1 1 1; visual mesh filename=package://overworld/models/adream/floor_hall.obj scale=1 1 1
Joints:
- joint base_to_floor: child adream_floor -> adream_floor_hall

Commit message: [Models] add adream FF

File: models/adream/adream.urdf (robot description, URDF)
Before this commit: robot adream, 9 links, 7 joints
Links:
- added link adream_gg_roof, mass .0; visual mesh filename=package://overworld/models/adream/adream_gg_roof.obj scale=1 1 1
- added link adream_window_h100_1, mass .0; visual mesh filename=package://overworld/models/adream/window_h100_1.obj scale=1 1 1
- added link adream_window_h100_2, mass .0; visual mesh filename=package://overworld/models/adream/window_h100_2.obj scale=1 1 1
- added link adream_window_h100_3, mass .0; visual mesh filename=package://overworld/models/adream/window_h100_3.obj scale=1 1 1
- added link ff_floor, mass .0; visual mesh filename=package://overworld/models/adream/ff_floor.obj scale=1 1 1
- added link ff_walls, mass .0; visual mesh filename=package://overworld/models/adream/ff_walls.obj scale=1 1 1
- added link guard_rail, mass .0; visual mesh filename=package://overworld/models/adream/guard_rail.obj scale=1 1 1
- added link hall_roof, mass .0; visual mesh filename=package://overworld/models/adream/hall_roof.obj scale=1 1 1

Commit message: [Models] fix adream urdf

File: models/adream/adream.urdf (robot description, URDF)
Before this commit: robot adream, 17 links, 7 joints
Joints:
- added joint base_to_adream_gg_roof: type fixed, parent adream_walls, child adream_gg_roof
- added joint base_to_adream_window_h100_1: type fixed, parent adream_walls, child adream_window_h100_1
- added joint base_to_adream_window_h100_2: type fixed, parent adream_walls, child adream_window_h100_2
- added joint base_to_adream_window_h100_3: type fixed, parent adream_walls, child adream_window_h100_3
- added joint base_to_ff_floor: type fixed, parent adream_walls, child ff_floor
- added joint base_to_ff_walls: type fixed, parent adream_walls, child ff_walls
- added joint base_to_floor_hall: type fixed, parent adream_walls, child adream_floor_hall
- added joint base_to_guard_rail: type fixed, parent adream_walls, child guard_rail
- added joint base_to_hall_roof: type fixed, parent adream_walls, child hall_roof
- joint base_to_floor: child adream_floor_hall -> adream_floor_expe

Commit message: add visual only entities

File: models/adream/adream.urdf (robot description, URDF)
Before this commit: robot adream, 17 links, 16 joints
Links:
- link adream_gg_roof: geometry visual mesh filename=package://overworld/models/adream/visual_only/adream_gg_roo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 scale=1 1 1
- link adream_window_h100_1: geometry visual mesh filename=package://overworld/models/adream/windows/window_h100_1.obj scale=1 1 1
- link adream_window_h100_2: geometry visual mesh filename=package://overworld/models/adream/windows/window_h100_2.obj scale=1 1 1
- link adream_window_h100_3: geometry visual mesh filename=package://overworld/models/adream/windows/window_h100_3.obj scale=1 1 1
- link adream_window_h10_1: geometry visual mesh filename=package://overworld/models/adream/windows/window_h10_1.stl scale=1 1 1
- link adream_window_h10_2: geometry visual mesh filename=package://overworld/models/adream/windows/window_h10_2.obj scale=1 1 1
- link adream_window_h20_1: geometry visual mesh filename=package://overworld/models/adream/windows/window_h20_1.obj scale=1 1 1
- link adream_window_h20_2: geometry visual mesh filename=package://overworld/models/adream/windows/window_h20_2.obj scale=1 1 1
- link adream_window_h20_3: geometry visual mesh filename=package://overworld/models/adream/windows/window_h20_3.obj scale=1 1 1
- link ff_floor: geometry visual mesh filename=package://overworld/models/adream/visual_only/ff_floor.obj scale=1 1 1
- link ff_walls: geometry visual mesh filename=package://overworld/models/adream/visual_only/ff_walls.obj scale=1 1 1
- link guard_rail: geometry visual mesh filename=package://overworld/models/adream/visual_only/guard_rail.obj scale=1 1 1
